File: hardware/discovery/audio.sch (KiCad schematic (older format))
At the start: 0 parts

Commit message: Discovery: Add audio DAC
Parts:
- added C10, C11: 1uF, Capacitors_SMD:C_0805, symbol Csmall
- added C6, C7, C8, C9: 0.1uF, Capacitors_SMD:C_0805, symbol C
- added J1: JACK_2P, symbol JACK_2P
- added U5: SGTL5000, Housings_DFN_QFN:UQFN-20-1EP_3x3mm_Pitch0.4mm, symbol SGTL5000
Connections:
- new net: C6.1, U5.5 (VAG)
- new net: J1.1, U5.4 (HP_L)
- new net: J1.2, U5.2 (HP_VGND)
- new net: J1.3, U5.1 (HP_R)
- new net: C7.2, U5.3 (VDDA)
- new net: C8.2, U5.12 (VDDIO)
- new net: C9.2, U5.20 (VDDD)
- new net: C11.2, U5.8 (LINE_IN_R)
- new net: C10.2, U5.9 (LINE_IN_L)
- new net 3V3: C7.1, C8.1, C9.1
- new net Audio_SCL: U5.19 (SCL)
- new net Audio_SDA: U5.18 (SDA)
- new net GND: C6.2, U5.21 (GND)
- new net I2S_DIN: U5.17 (I2S_DIN)
- new net I2S_DOUT: U5.16 (I2S_DOUT)
- new net I2S_LRCLK: U5.14 (I2S_LRCLK)
- new net I2S_MCLK: U5.13 (I2S_MCLK)
- new net I2S_SCLK: U5.15 (I2S_SCLK)
- new net LINE_IN_L: C10.1
- new net LINE_IN_R: C11.1
Changed lines of the file:
@@
 Comment4 ""
 $EndDescr
+Text GLabel 5150 2900 0    60   Input ~ 0
+Audio_SDA
+Text GLabel 5150 3050 0    60   Input ~ 0
+Audio_SCL
+Text GLabel 5150 3300 0    60   Input ~ 0
+I2S_MCLK
+Text GLabel 5150 3450 0    60   Input ~ 0
+I2S_SCLK
+Text GLabel 5150 3600 0    60   Input ~ 0
+I2S_LRCLK
+Text GLabel 5150 3750 0    60   Input ~ 0
+I2S_DIN
+Text GLabel 5150 3900 0    60   Input ~ 0
+I2S_DOUT
+Text GLabel 5250 2050 0    60   Input ~ 0
+3V3
+Wire Wire Line
+	5150 4250 5100 4250
+Wire Wire Line
+	5100 4250 5100 4450
+$Comp
+L GND #PWR023
+U 1 1 585E79AD
+P 5100 4450
+F 0 "#PWR023" H 5100 4450 30  0001 C CNN
+F 1 "GND" H 5100 4380 30  0001 C CNN
+F 2 "" H 5100 4450 60  0001 C CNN
+F 3 "" H 5100 4450 60  0001 C CNN
+	1    5100 4450
+	1    0    0    -1
+$EndComp
+$Comp
+L C C6
+U 1 1 585E7B78
+P 4750 4300
+F 0 "C6" H 4750 4400 40  0000 L CNN
+F 1 "0.1uF" H 4756 4215 40  0000 L CNN
+F 2 "Capacitors_SMD:C_0805" H 4788 4150 30  0001 C CNN
+F 3 "" H 4750 4300 60  0000 C CNN
+	1    4750 4300
+	1    0    0    -1
+$EndComp
+$Comp
+L GND #PWR024
+U 1 1 585E7BA3
+P 4750 4500
+F 0 "#PWR024" H 4750 4500 30  0001 C CNN
+F 1 "GND" H 4750 4430 30  0001 C CNN
+F 2 "" H 4750 4500 60  0001 C CNN
+F 3 "" H 4750 4500 60  0001 C CNN
+	1    4750 4500
+	1    0    0    -1
+$EndComp
+Wire Wire Line
+	5150 4100 4750 4100
+$Comp
+L JACK_2P J1
+U 1 1 585E7EFF
+P 7500 3650
+F 0 "J1" H 7150 3450 60  0000 C CNN
+F 1 "JACK_2P" H 7350 3900 60  0000 C CNN
+F 2 "" H 7500 3650 60  0001 C CNN
+F 3 "" H 7500 3650 60  0000 C CNN
+	1    7500 3650
+	-1   0    0    1
+$EndComp
+Wire Wire Line
+	6400 3500 7050 3500
+Wire Wire Line
+	7050 3500 7050 3550
+Wire Wire Line
+	6400 3650 6800 3650
+Wire Wire Line
+	6800 3650 6800 3800
+Wire Wire Line
+	6800 3800 7050 3800
+Wire Wire Line
+	7050 3650 6900 3650
+Wire Wire Line
+	6900 3650 6900 3750
+Wire Wire Line
+	6900 3750 6400 3750
+Wire Wire Line
+	6400 3750 6400 3800
+$Comp
+L C C7
+U 1 1 585E8504
+P 5550 2300
+F 0 "C7" H 5550 2400 40  0000 L CNN
+F 1 "0.1uF" H 5556 2215 40  0000 L CNN
+F 2 "Capacitors_SMD:C_0805" H 5588 2150 30  0001 C CNN
+F 3 "" H 5550 2300 60  0000 C CNN
+	1    5550 2300
+	1    0    0    -1
+$EndComp
+$Comp
+L C C8
+U 1 1 585E857A
+P 5800 2300
+F 0 "C8" H 5800 2400 40  0000 L CNN
+F 1 "0.1uF" H 5806 2215 40  0000 L CNN
+F 2 "Capacitors_SMD:C_0805" H 5838 2150 30  0001 C CNN
+F 3 "" H 5800 2300 60  0000 C CNN
+	1    5800 2300
+	1    0    0    -1
+$EndComp
+$Comp
+L C C9
+U 1 1 585E859F
+P 6050 2300
+F 0 "C9" H 6050 2400 40  0000 L CNN
+F 1 "0.1uF" H 6056 2215 40  0000 L CNN
+F 2 "Capacitors_SMD:C_0805" H 6088 2150 30  0001 C CNN
+F 3 "" H 6050 2300 60  0000 C CNN
+	1    6050 2300
+	1    0    0    -1
+$EndComp
+$Comp
+L SGTL5000 U5
+U 1 1 585E883F
+P 5400 2800
+F 0 "U5" H 5300 3050 60  0000 C CNN
+F 1 "SGTL5000" H 5750 1250 60  0000 C CNN
+F 2 "Housings_DFN_QFN:UQFN-20-1EP_3x3mm_Pitch0.4mm" H 5400 2750 60  0001 C CNN
+F 3 "" H 5400 2750 60  0001 C CNN
+	1    5400 2800
+	1    0    0    -1
+$EndComp
+Wire Wire Line
+	6050 2100 6050 2050
+Wire Wire Line
+	6050 2050 5250 2050
+Wire Wire Line
+	5550 2100 5550 2050
+Connection ~ 5550 2050
+Wire Wire Line
+	5800 2100 5800 2050
+Connection ~ 5800 2050
+$Comp
+L Csmall C10
+U 1 1 585E8C6B
+P 6650 2900
+F 0 "C10" V 6700 2800 30  0000 L CNN
+F 1 "1uF" V 6700 2950 30  0000 L CNN
+F 2 "Capacitors_SMD:C_0805" H 6650 2900 60  0001 C CNN
+F 3 "" H 6650 2900 60  0000 C CNN
+	1    6650 2900
+	0    1    1    0
+$EndComp
+$Comp
+L Csmall C11
+U 1 1 585E8E3F
+P 6650 3050
+F 0 "C11" V 6700 2950 30  0000 L CNN
+F 1 "1uF" V 6700 3100 30  0000 L CNN
+F 2 "Capacitors_SMD:C_0805" H 6650 3050 60  0001 C CNN
+F 3 "" H 6650 3050 60  0000 C CNN
+	1    6650 3050
+	0    1    1    0
+$EndComp
+Wire Wire Line
+	6550 2900 6400 2900
+Wire Wire Line
+	6550 3050 6400 3050
+Wire Wire Line
+	6750 2900 6950 2900
+Wire Wire Line
+	6750 3050 6950 3050
+Text GLabel 6950 2900 2    60   Input ~ 0
+LINE_IN_L
+Text GLabel 6950 3050 2    60   Input ~ 0
+LINE_IN_R
 $EndSCHEMATC

Commit message: Discovery: Add audio jacks
Parts:
- removed J1: JACK_2P, symbol JACK_2P
- added HP_OUT1, LINE_IN1: 3.5_audio_jack, stm32f4-disco:lumberg_3.5_audio_jack_1503_02, symbol 3.5_audio_jack
Connections:
- net GND: now also LINE_IN1.2 (SLEEVE)
- net at U5.4 (HP_L): now also HP_OUT1.1 (TIP)
- net at U5.2 (HP_VGND): now also HP_OUT1.2 (SLEEVE)
- net at U5.1 (HP_R): now also HP_OUT1.3 (RING)
- net LINE_IN_L: no longer names the net of C10.1
- net LINE_IN_L: now also LINE_IN1.1 (TIP)
- net LINE_IN_R: no longer names the net of C11.1
- net LINE_IN_R: now also LINE_IN1.3 (RING)
Changed lines of the file:
@@
 Wire Wire Line
 	5150 4100 4750 4100
-$Comp
-L JACK_2P J1
-U 1 1 585E7EFF
-P 7500 3650
-F 0 "J1" H 7150 3450 60  0000 C CNN
-F 1 "JACK_2P" H 7350 3900 60  0000 C CNN
-F 2 "" H 7500 3650 60  0001 C CNN
-F 3 "" H 7500 3650 60  0000 C CNN
-	1    7500 3650
-	-1   0    0    1
-$EndComp
 Wire Wire Line
-	6400 3500 7050 3500
+	6400 3500 7375 3500
 Wire Wire Line
-	7050 3500 7050 3550
-Wire Wire Line
-	6400 3650 6800 3650
-Wire Wire Line
-	6800 3650 6800 3800
-Wire Wire Line
-	6800 3800 7050 3800
-Wire Wire Line
-	7050 3650 6900 3650
-Wire Wire Line
-	6900 3650 6900 3750
-Wire Wire Line
-	6900 3750 6400 3750
-Wire Wire Line
-	6400 3750 6400 3800
+	6400 3650 7375 3650
 $Comp
 L C C7
@@
 	6550 3050 6400 3050
 Wire Wire Line
-	6750 2900 6950 2900
+	6750 2900 7375 2900
 Wire Wire Line
-	6750 3050 6950 3050
-Text GLabel 6950 2900 2    60   Input ~ 0
-LINE_IN_L
-Text GLabel 6950 3050 2    60   Input ~ 0
-LINE_IN_R
+	6750 3050 7375 3050
+$Comp
+L 3.5_audio_jack HP_OUT1
+U 1 1 5863AC9E
+P 7750 4025
+F 0 "HP_OUT1" H 7825 3400 60  0000 C CNN
+F 1 "3.5_audio_jack" H 7750 4025 60  0001 C CNN
+F 2 "stm32f4-disco:lumberg_3.5_audio_jack_1503_02" H 7750 4025 60  0001 C CNN
+F 3 "" H 7750 4025 60  0001 C CNN
+	1    7750 4025
+	-1   0    0    1
+$EndComp
+Wire Wire Line
+	6400 3800 7375 3800
+$Comp
+L 3.5_audio_jack LINE_IN1
+U 1 1 5863B129
+P 7750 3425
+F 0 "LINE_IN1" H 7825 2800 60  0000 C CNN
+F 1 "3.5_audio_jack" H 7600 2800 60  0001 C CNN
+F 2 "stm32f4-disco:lumberg_3.5_audio_jack_1503_02" H 7750 3425 60  0001 C CNN
+F 3 "" H 7750 3425 60  0001 C CNN
+	1    7750 3425
+	-1   0    0    1
+$EndComp
+$Comp
+L GND #PWR026
+U 1 1 5863B3F7
+P 7325 3275
+F 0 "#PWR026" H 7325 3275 30  0001 C CNN
+F 1 "GND" H 7325 3205 30  0001 C CNN
+F 2 "" H 7325 3275 60  0001 C CNN
+F 3 "" H 7325 3275 60  0001 C CNN
+	1    7325 3275
+	1    0    0    -1
+$EndComp
+Wire Wire Line
+	7375 3200 7325 3200
+Wire Wire Line
+	7325 3200 7325 3275
 $EndSCHEMATC
