File: hardware/discovery/poss_discovery.sch (KiCad schematic (older format))
At the start: 35 parts, among them SW1 SW_PUSH, SW10 SW_PUSH, SW11 SW_PUSH, SW12 SW_PUSH, SW13 SW_PUSH, SW14 SW_PUSH, SW15 SW_PUSH, SW16 SW_PUSH, SW18 SW_PUSH, SW19 SW_PUSH, SW2 SW_PUSH, SW20 SW_PUSH, SW21 SW_PUSH, SW22 SW_PUSH, SW3 SW_PUSH, SW4 SW_PUSH, SW5 SW_PUSH, SW6 SW_PUSH, SW7 SW_PUSH, SW8 SW_PUSH, SW9 SW_PUSH, U1 STM32F4_DISCO_Header, U6 encoder_and_switch, U7 encoder_and_switch

Commit message: Discovery: Update TODO list
Other:
- note added: "TODO:\n - BOOT line \n and DFU mode"
- note removed: "TODO:\n - Debug port\n - Encoders capa\n - VBAT sensing\n - BOOT line \n and DFU mode"
Changed lines of the file:
@@
 F1 "audio.sch" 60
 $EndSheet
-Text Notes 8950 5850 0    157  ~ 0
-TODO:\n - Debug port\n - Encoders capa\n - VBAT sensing\n - BOOT line \n    and DFU mode
+Text Notes 8950 4900 0    157  ~ 0
+TODO:\n - BOOT line \n    and DFU mode
 Text GLabel 6800 3750 0    60   Input ~ 0
 WAKEUP

Commit message: Discovery: Restart from RevA
Parts:
- removed C30, C31, C32, C33: 0,1uF, Capacitors_SMD:C_0805, symbol C
- removed R16, R17, R18, R19: 27K, Resistors_SMD:R_0805, symbol R
- removed U1: STM32F4_DISCO_Header, stm32f4-disco:STM32F4-DISCO-HEADERS-SMD, symbol STM32F4_DISCO_Header
- removed U6, U7: encoder_and_switch, stm32f4-disco:encoder_EC12D, symbol encoder_and_switch
- added D1, D10, D11, D12, D13, D14, D15, D16, D17, D18, D19, D2, D20, D21, D22, D23, D24, D25, D3, D4, D5, D6, D7, D8, D9: LED, LEDs:LED_0805, symbol LED
- added J1, J5: HEADER_2, Pin_Headers:Pin_Header_Straight_2x01, symbol HEADER_2
- added J2, J3: HEADER_25x2, Pin_Headers:Pin_Header_Straight_2x25, symbol HEADER_25x2
- added RV1, RV2: POT, Potentiometers:Potentiometer_WirePads_Small, symbol POT-RESCUE-poss_discovery
- added SW17: SW_PUSH, Buttons_Switches_SMD:SW_SPST_B3SL-1002P, symbol SW_PUSH
Connections:
- net WAKEUP is gone; now on net GND: Play1.2, Play2.2, SW1.2, SW10.2, SW11.2, SW12.2, SW13.2, SW14.2, SW15.2, SW16.2, SW18.2, SW19.2, SW2.2, SW20.2, SW21.2, SW22.2, SW3.2, SW4.2, SW5.2, SW6.2, SW7.2, SW8.2, SW9.2, Write1.2
- net Audio_Reset: now also J3.20
- net Audio_SCL: now also J3.27
- net Audio_SDA: now also J3.32
- net B1: now also J3.42
- net B10: now also J3.41
- net B11: now also J3.39
- net B12: now also J3.38
- net B13: now also J3.35
- net B14: now also J3.25
- net B15: now also J3.24
- net B16: now also J3.19
- net B2: now also J3.40
- net B3: now also J3.37
- net B4: now also J3.31
- net B5: now also J3.26
- net B6: now also J3.23
- net B7: now also J3.22
- net B8: now also J3.17
- net B9: now also J3.28
- net COL1: now also D1.2 (K), D2.2 (K), D3.2 (K), D4.2 (K), D5.2 (K), J3.3
- net COL2: now also D10.2 (K), D6.2 (K), D7.2 (K), D8.2 (K), D9.2 (K), J3.9
- net COL3: now also D11.2 (K), D12.2 (K), D13.2 (K), D14.2 (K), D15.2 (K), J2.38
- net COL4: now also D16.2 (K), D17.2 (K), D18.2 (K), D19.2 (K), D20.2 (K), J2.41
- net COL5: now also D21.2 (K), D22.2 (K), D23.2 (K), D24.2 (K), D25.2 (K), J2.44
- net CS_I2C/SPI: now also J3.36
- net FX: now also J2.7
- net GND: now also J1.1, J1.2, J2.1, J2.2, J2.27, J2.45, J2.49, J2.50, J3.1, J3.2, J3.49, J3.50, J5.1, J5.2, RV1.3, RV2.3, SW17.2
- net I2S3_MCK: now also J3.4
- net I2S3_SCK: now also J3.13
- net I2S3_SD: now also J3.15
- net I2S3_WS: now also J2.36
- net MEMS_INT1: now also J3.33
- net MEMS_INT2: now also J3.34
- net BA renamed BF2
- net BF2: now also J2.42
- net BB renamed BF3
- net BF3: now also J2.12
- net BC renamed BF4
- net BF4: now also J2.11
- net BD renamed BF5
- net BF5: now also J2.10
- net BE renamed BPM
- net BPM: now also J2.9
- net Play renamed PD0
- net PD0: now also J3.16
- net Write renamed PD2
- net PD2: now also J3.18
- new net 3V: J3.45, J3.46, RV1.1, RV2.1
- new net 5V: J3.47, J3.48
- new net BF1: J2.43, SW17.1
- new net BOOT0: J3.29
- new net NC: J2.4
- new net NRTS: J2.46
- new net PA0: J2.40
- new net PA1: J2.39, RV1.2
- new net PA13: J3.10
- new net PA14: J3.11
- new net PA15: D13.1 (A), D18.1 (A), D23.1 (A), D3.1 (A), D8.1 (A), J3.12
- new net PA3: J2.37, RV2.2
- new net PA5: J2.35
- new net PA6: J2.34
- new net PA7: J2.33
- new net PA8: D10.1 (A), D15.1 (A), D20.1 (A), D25.1 (A), D5.1 (A), J3.7
- new net PA9: J3.8
- new net PB0: J2.30
- new net PB1: J2.29
- new net PB10: J2.18
- new net PB11: J2.15
- new net PB12: J2.16
- new net PB13: J2.13
- new net PB14: J2.14
- new net PB2: J2.28
- new net PC11: D14.1 (A), D19.1 (A), D24.1 (A), D4.1 (A), D9.1 (A), J3.14
- new net PC4: J2.32
- new net PC5: J2.31
- new net PC8: D12.1 (A), D17.1 (A), D2.1 (A), D22.1 (A), D7.1 (A), J3.5
- new net PC9: D1.1 (A), D11.1 (A), D16.1 (A), D21.1 (A), D6.1 (A), J3.6
- new net PD12: J2.8
- new net PD13: J2.5
- new net PD14: J2.6
- new net PD15: J2.3
- new net PD5: J3.21
- new net PE10: J2.24
- new net PE11: J2.21
- new net PE12: J2.22
- new net PE13: J2.19
- new net PE14: J2.20
- new net PE15: J2.17
- new net PE7: J2.25
- new net PE8: J2.26
- new net PE9: J2.23
- new net PH0: J3.43
- new net PH1: J3.44
- new net VDD: J2.47, J2.48
- new net VDD2: J3.30
Other:
- note added: "Known Problems:"
- note removed: "TODO:\n - BOOT line \n and DFU mode"
