File: hardware/discovery/wnm_discovery.sch (KiCad schematic (older format))
At the start: 56 parts, among them J1 HEADER_2, J2 HEADER_25x2, J3 HEADER_25x2, J5 HEADER_2, SW1 SW_PUSH, SW10 SW_PUSH, SW11 SW_PUSH, SW12 SW_PUSH, SW13 SW_PUSH, SW14 SW_PUSH, SW15 SW_PUSH, SW16 SW_PUSH, SW17 SW_PUSH, SW18 SW_PUSH, SW19 SW_PUSH, SW2 SW_PUSH, SW20 SW_PUSH, SW21 SW_PUSH, SW22 SW_PUSH, SW3 SW_PUSH, SW4 SW_PUSH, SW5 SW_PUSH, SW6 SW_PUSH, SW7 SW_PUSH, SW8 SW_PUSH, SW9 SW_PUSH

Commit message: HW: Update discovery with new UI design (encoders, screen, buttons layout)
Parts:
- removed D1, D10, D11, D12, D13, D14, D15, D16, D17, D18, D19, D2, D20, D21, D22, D23, D24, D25, D3, D4, D5, D6, D7, D8, D9: LED, LEDs:LED_0805, symbol LED
- removed J1, J5: HEADER_2, Pin_Headers:Pin_Header_Straight_2x01, symbol HEADER_2
- removed J2, J3: HEADER_25x2, Pin_Headers:Pin_Header_Straight_2x25, symbol HEADER_25x2
- removed RV1, RV2: POT, Potentiometers:Potentiometer_WirePads_Small, symbol POT-RESCUE-poss_discovery
- removed SW17: SW_PUSH, Buttons_Switches_SMD:SW_SPST_B3SL-1002P, symbol SW_PUSH
- added C30, C31, C32, C33: 0,1uF, Capacitors_SMD:C_0805, symbol C
- added R16, R17, R18, R19: 27K, Resistors_SMD:R_0805, symbol R
- added U6, U7: encoder_and_switch, POSS:encoder_EC12D, symbol encoder_and_switch
Connections:
- net labels added: BA, BB, BC, BD, BE, ENC_1_A, ENC_1_B, ENC_1_SW, ENC_2_A, ENC_2_B, ENC_2_SW, WAKEUP
- net labels removed: 3V, 5V, Audio_Reset, Audio_SCL, Audio_SDA, BF1, BF2, BF3, BF4, BF5, BOOT0, BP7, BPM, COL1, COL2, COL3, COL4, COL5, CS_I2C/SPI, I2S3_MCK, I2S3_SCK, I2S3_SD, I2S3_WS, MEMS_INT1, MEMS_INT2, NC, NRTS, PA0, PA1, PA10, PA13, PA14, PA15, PA2, PA3, PA4, PA5, PA6, PA7, PA8, PA9, PB0, PB1, PB10, PB11, PB12, PB13, PB14, PB15, PB2, PB3, PB4, PB5, PB6, PB8, PB9, PC0, PC1, PC10, PC11, PC12, PC13, PC14, PC15, PC2, PC3, PC4, PC5, PC6, PC7, PC8, PC9, PD0, PD1, PD10, PD11, PD12, PD13, PD14, PD15, PD2, PD3, PD4, PD5, PD6, PD7, PD8, PD9, PE0, PE1, PE10, PE11, PE12, PE13, PE14, PE15, PE2, PE3, PE4, PE5, PE6, PE7, PE8, PE9, PH0, PH1, POT1, POT2, ROW1, ROW2, ROW3, ROW4, ROW5, SPI1_MISO, SPI1_MOSI, SPI1_SCK, STM_LED2, STM_LED3, STM_LED4, STM_LED_1, STM_USER_BTN, SWCLK, SWDIO, USB_Over_I, VDD, VDD2, Vbus_FS
- wire segments 173 -> 4
Other:
- note added: "TODO:"
- note removed: "Known Problems:"
- moved on the sheet: Play1, Play2, SW1, SW10, SW11, SW12, SW13, SW14, SW15, SW16, SW18, SW19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

Commit message: HW: Use a different MCU pins for the discovery board
This simplifies the PCB layout.
Parts:
- C30, C31, C32, C33: symbol C -> C-RESCUE-wnm_discovery
- R16, R17, R18, R19: symbol R -> R-RESCUE-wnm_discovery
Changed lines of the file:
@@
 EESchema Schematic File Version 2
+LIBS:wnm_discovery-rescue
 LIBS:power
 LIBS:device
@@
 LIBS:microchip_pic12mcu
 LIBS:microchip_pic16mcu
-LIBS:microchip1
 LIBS:msp430
 LIBS:nxp_armmcu
@@
 LIBS:relays
 LIBS:sensors
-LIBS:special
 LIBS:stm8
 LIBS:stm32
@@
 B16
 $Sheet
-S 2400 650  1400 1100
+S 2550 650  1400 1100
 U 585DBE08
 F0 "Micro-Controller" 60
@@
 $EndSheet
 $Sheet
-S 4050 650  1450 1050
+S 4750 800  1450 1050
 U 585D6FEE
 F0 "LED_Matrix" 60
@@
 ENC_1_B
 $Comp
-L GND #PWR01
+L GND-RESCUE-wnm_discovery #PWR01
 U 1 1 586532D8
 P 4950 7050
@@
 $EndComp
 $Comp
-L GND #PWR02
+L GND-RESCUE-wnm_discovery #PWR02
 U 1 1 58653337
 P 2200 7050
@@
 	8000 3750 8000 5700
 $Comp
-L R R16
+L R-RESCUE-wnm_discovery R16
 U 1 1 58664AEC
 P 1700 7050
@@
 $EndComp
 $Comp
-L C C30
+L C-RESCUE-wnm_discovery C30
 U 1 1 58664DFD
 P 1450 7250
@@
 $EndComp
 $Comp
-L GND #PWR03
+L GND-RESCUE-wnm_discovery #PWR03
 U 1 1 58664E6F
 P 1450 7450
@@
 $EndComp
 $Comp
-L R R17
+L R-RESCUE-wnm_discovery R17
 U 1 1 586652D6
 P 2700 7050
@@
 $EndComp
 $Comp
-L C C31
+L C-RESCUE-wnm_discovery C31
 U 1 1 586655E8
 P 2950 7250
@@
 $EndComp
 $Comp
-L GND #PWR04
+L GND-RESCUE-wnm_discovery #PWR04
 U 1 1 5866566D
 P 2950 7450
@@
 ENC_2_B
 $Comp
-L R R19
+L R-RESCUE-wnm_discovery R19
 U 1 1 58665F22
 P 5450 7050
@@
 $EndComp
 $Comp
-L C C33
+L C-RESCUE-wnm_discovery C33
 U 1 1 58665F28
 P 5700 7250
@@
 $EndComp
 $Comp
-L GND #PWR05
+L GND-RESCUE-wnm_discovery #PWR05
 U 1 1 58665F2E
 P 5700 7450
@@
 ENC_2_A
 $Comp
-L R R18
+L R-RESCUE-wnm_discovery R18
 U 1 1 58666537
 P 4450 7050
@@
 $EndComp
 $Comp
-L C C32
+L C-RESCUE-wnm_discovery C32
 U 1 1 5866653D
 P 4200 7250
@@
 $EndComp
 $Comp
-L GND #PWR06
+L GND-RESCUE-wnm_discovery #PWR06
 U 1 1 58666543
 P 4200 7450

Commit message: HW:Update revision of the discovery board
Changed lines of the file:
@@
 encoding utf-8
 Sheet 1 3
-Title "Wee Noise Maker - Mk-I"
+Title "Wee Noise Maker - Discovery"
 Date ""
-Rev "A"
+Rev "B"
 Comp "Fabien Chouteau"
 Comment1 ""
@@
 $EndSheet
 $Sheet
-S 4750 800  1450 1050
+S 4000 650  1450 1050
 U 585D6FEE
 F0 "LED_Matrix" 60
