File: hardware/Mk-I/poss_mk_1.kicad_pcb (KiCad board)
At the start: 2 copper layers, 96.5 x 66 mm, 118 parts, among them CON1 USB-MICRO-B, SW1 SW_PUSH, SW10 SW_PUSH, SW11 SW_PUSH, SW12 SW_PUSH, SW13 SW_PUSH, SW14 SW_PUSH, SW15 SW_PUSH, SW16 SW_PUSH, SW18 SW_PUSH, SW19 SW_PUSH, SW2 SW_PUSH, SW20 SW_PUSH, SW21 SW_PUSH, SW22 SW_PUSH, SW3 SW_PUSH, SW4 SW_PUSH, SW5 SW_PUSH, SW6 SW_PUSH, SW7 SW_PUSH, SW8 SW_PUSH, SW9 SW_PUSH, U10 STM32_SWD_Connector, U2 MCP73831, U3 BD33IA5, U4 STM32F407VG, U5 SGTL5000, U6 encoder_and_switch, U7 encoder_and_switch, U8 MOLEX_microSD_47219-2001, U9 SSD1306, X1 CRYSTAL

Commit message: Mk-I: A couple of fixes in silkscreen
Other:
- board text removed: "RevB"
Changed lines of the file:
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@@
     (area 79.934999 78.664999 176.605001 144.855001)
     (thickness 1.6)
-    (drawings 93)
+    (drawings 92)
     (tracks 1923)
     (zones 0)
@@
   (module POSS:lumberg_3.5_audio_jack_1503_02 (layer B.Cu)
     (at 174.3456 83 180)
-    (fp_text reference HP_OUT1 (at 0 -0.5 180) (layer B.SilkS)
+    (fp_text reference HP_OUT1 (at 0 -0.5 180) (layer B.SilkS) hide
       (effects (font (size 1 1) (thickness 0.15)) (justify mirror))
     )
@@
   (module POSS:lumberg_3.5_audio_jack_1503_02 (layer B.Cu)
     (at 82.1436 91.2876)
-    (fp_text reference LINE_IN1 (at 0 -0.5) (layer B.SilkS)
+    (fp_text reference LINE_IN1 (at 0 -0.5) (layer B.SilkS) hide
       (effects (font (size 1 1) (thickness 0.15)) (justify mirror))
     )
@@
   (gr_line (start 123.8504 104.14) (end 113.0554 104.14) (angle 90) (layer F.SilkS) (width 0.2))
   (gr_line (start 161.9504 104.14) (end 123.8504 104.14) (angle 90) (layer F.SilkS) (width 0.2))
-  (gr_text RevB (at 170.688 143.002) (layer B.SilkS)
-    (effects (font (size 1.5 1.5) (thickness 0.3)) (justify mirror))
-  )
   (gr_line (start 145.288 127.762) (end 145.288 126.238) (angle 90) (layer F.SilkS) (width 0.2))
   (gr_line (start 151.892 127.762) (end 151.892 126.238) (angle 90) (layer F.SilkS) (width 0.2))

Commit message: MK-I : Decrease mask clearance to ~3mil
Other:
- rule pad_to_mask_clearance: 0.2 -> 0.08
Changed lines of the file:
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@@
     (pad_size 1.524 1.524)
     (pad_drill 0.762)
-    (pad_to_mask_clearance 0.2)
+    (pad_to_mask_clearance 0.08)
     (aux_axis_origin 80.01 144.78)
     (visible_elements 7FFEEE7F)
