File: hardware/Mk-I/button_matrix.sch (KiCad schematic (older format))
At the start: 33 parts, among them SW1 EVQ-Q2S02W, SW10 EVQ-Q2S02W, SW11 EVQ-Q2S02W, SW12 EVQ-Q2S02W, SW13 EVQ-Q2S02W, SW14 EVQ-Q2S02W, SW15 EVQ-Q2S02W, SW16 EVQ-Q2S02W, SW2 EVQ-Q2S02W, SW20 EVQ-Q2S02W, SW21 EVQ-Q2S02W, SW22 EVQ-Q2S02W, SW3 EVQ-Q2S02W, SW4 EVQ-Q2S02W, SW5 EVQ-Q2S02W, SW6 EVQ-Q2S02W, SW7 EVQ-Q2S02W, SW8 EVQ-Q2S02W, SW9 EVQ-Q2S02W, U6 EC12D1524403, U7 EC12D1524403

Commit message: HW: Finish rev-D layout
Parts:
- removed R16, R17, R18, R19: 27K, Resistors_SMD:R_0805, symbol R-RESCUE-wnm_mk_1
Connections:
- net ENC_1_A: now also U6.1 (A)
- net ENC_1_B: now also U6.2 (B)
- net ENC_2_A: now also U7.1 (A)
- net ENC_2_B: now also U7.2 (B)
- net GND: now also U6.6 (shield), U7.6 (shield)
Changed lines of the file:
@@
 U 1 1 59ED2A61
 P 3100 5100
-F 0 "U6" H 2850 4900 60  0000 C CNN
-F 1 "EC12D1524403" H 3450 4950 60  0000 C CNN
+F 0 "U6" H 2900 4950 60  0000 C CNN
+F 1 "EC12D1524403" H 3750 4950 60  0000 C CNN
 F 2 "POSS:encoder_EC12D" H 3100 5100 60  0001 C CNN
 F 3 "" H 3100 5100 60  0001 C CNN
@@
 U 1 1 59ED2A68
 P 5850 5100
-F 0 "U7" H 5600 4900 60  0000 C CNN
-F 1 "EC12D1524403" H 6200 4950 60  0000 C CNN
+F 0 "U7" H 5650 4950 60  0000 C CNN
+F 1 "EC12D1524403" H 6550 4900 60  0000 C CNN
 F 2 "POSS:encoder_EC12D" H 5850 5100 60  0001 C CNN
 F 3 "" H 5850 5100 60  0001 C CNN
@@
 $EndComp
 $Comp
-L R-RESCUE-wnm_mk_1 R16
-U 1 1 59ED2A81
-P 2600 5800
-F 0 "R16" V 2680 5800 40  0000 C CNN
-F 1 "27K" V 2607 5801 40  0000 C CNN
-F 2 "Resistors_SMD:R_0805" V 2530 5800 30  0001 C CNN
-F 3 "" H 2600 5800 30  0000 C CNN
-	1    2600 5800
-	0    1    1    0
-$EndComp
-$Comp
 L C-RESCUE-wnm_mk_1 C30
 U 1 1 59ED2A88
@@
 	1    2350 6200
 	1    0    0    -1
-$EndComp
-$Comp
-L R-RESCUE-wnm_mk_1 R17
-U 1 1 59ED2A95
-P 3600 5800
-F 0 "R17" V 3680 5800 40  0000 C CNN
-F 1 "27K" V 3607 5801 40  0000 C CNN
-F 2 "Resistors_SMD:R_0805" V 3530 5800 30  0001 C CNN
-F 3 "" H 3600 5800 30  0000 C CNN
-	1    3600 5800
-	0    1    1    0
 $EndComp
 $Comp
@@
 ENC_2_B
 $Comp
-L R-RESCUE-wnm_mk_1 R19
-U 1 1 59ED2AAA
-P 6350 5800
-F 0 "R19" V 6430 5800 40  0000 C CNN
-F 1 "27K" V 6357 5801 40  0000 C CNN
-F 2 "Resistors_SMD:R_0805" V 6280 5800 30  0001 C CNN
-F 3 "" H 6350 5800 30  0000 C CNN
-	1    6350 5800
-	0    1    1    0
-$EndComp
-$Comp
 L C-RESCUE-wnm_mk_1 C33
 U 1 1 59ED2AB1
@@
 Text GLabel 5100 5800 0    60   Input ~ 0
 ENC_2_A
-$Comp
-L R-RESCUE-wnm_mk_1 R18
-U 1 1 59ED2ABF
-P 5350 5800
-F 0 "R18" V 5430 5800 40  0000 C CNN
-F 1 "27K" V 5357 5801 40  0000 C CNN
-F 2 "Resistors_SMD:R_0805" V 5280 5800 30  0001 C CNN
-F 3 "" H 5350 5800 30  0000 C CNN
-	1    5350 5800
-	0    1    1    0
-$EndComp
 $Comp
 L C-RESCUE-wnm_mk_1 C32
@@
 Wire Wire Line
 	5450 4700 4050 4700
+$Comp
+L GND-RESCUE-wnm_mk_1 #PWR041
+U 1 1 59F35037
+P 3100 4900
+F 0 "#PWR041" H 3100 4900 30  0001 C CNN
+F 1 "GND" H 3100 4830 30  0001 C CNN
+F 2 "" H 3100 4900 60  0001 C CNN
+F 3 "" H 3100 4900 60  0001 C CNN
+	1    3100 4900
+	-1   0    0    1
+$EndComp
+$Comp
+L GND-RESCUE-wnm_mk_1 #PWR042
+U 1 1 59F3537B
+P 5850 4900
+F 0 "#PWR042" H 5850 4900 30  0001 C CNN
+F 1 "GND" H 5850 4830 30  0001 C CNN
+F 2 "" H 5850 4900 60  0001 C CNN
+F 3 "" H 5850 4900 60  0001 C CNN
+	1    5850 4900
+	-1   0    0    1
+$EndComp
+Wire Wire Line
+	6100 5800 6600 5800
+Wire Wire Line
+	5600 5800 5100 5800
+Wire Wire Line
+	3850 5800 3350 5800
+Wire Wire Line
+	2850 5800 2350 5800
 $EndSCHEMATC

Commit message: HW: rev D production files
Parts:
- C30, C31: value 0.1uF -> 10nF
Changed lines of the file:
@@
 P 2350 6000
 F 0 "C30" H 2350 6100 40  0000 L CNN
-F 1 "0.1uF" H 2356 5915 40  0000 L CNN
+F 1 "10nF" H 2356 5915 40  0000 L CNN
 F 2 "Capacitors_SMD:C_0805" H 2388 5850 30  0001 C CNN
 F 3 "" H 2350 6000 60  0000 C CNN
@@
 P 3850 6000
 F 0 "C31" H 3850 6100 40  0000 L CNN
-F 1 "0.1uF" H 3856 5915 40  0000 L CNN
+F 1 "10nF" H 3856 5915 40  0000 L CNN
 F 2 "Capacitors_SMD:C_0805" H 3888 5850 30  0001 C CNN
 F 3 "" H 3850 6000 60  0000 C CNN
