File: hardware/Mk-I/led_matrix.sch (KiCad schematic (older format))
At the start: 34 parts, among them U9 SSD1306

Commit message: HW: Major change of layout...
Parts:
- removed D20, D21, D22, D23, D24: 150060GS75000, LEDs:LED_0805, symbol LED
- removed D25: 150060RS75000, LEDs:LED_0805, symbol LED
- removed R9: 330, Resistors_SMD:R_0805, symbol R-RESCUE-wnm_mk_1
Changed lines of the file:
@@
 $Descr A4 11693 8268
 encoding utf-8
-Sheet 4 5
+Sheet 4 6
 Title "Wee Noise Maker - Mk-I"
 Date ""
@@
 $EndComp
 $Comp
-L LED D25
-U 1 1 585D8AD0
-P 3300 5250
-AR Path="/585D8AD0" Ref="D25"  Part="1"
-AR Path="/585D6FEE/585D8AD0" Ref="D25"  Part="1"
-F 0 "D25" H 3300 5350 50  0000 C CNN
-F 1 "150060RS75000" H 3300 5150 50  0000 C CNN
-F 2 "LEDs:LED_0805" H 3300 5250 50  0001 C CNN
-F 3 "" H 3300 5250 50  0000 C CNN
-	1    3300 5250
-	1    0    0    -1
-$EndComp
-$Comp
-L LED D20
-U 1 1 585D8ADE
-P 3300 3500
-AR Path="/585D8ADE" Ref="D20"  Part="1"
-AR Path="/585D6FEE/585D8ADE" Ref="D20"  Part="1"
-F 0 "D20" H 3300 3600 50  0000 C CNN
-F 1 "150060GS75000" H 3300 3400 50  0000 C CNN
-F 2 "LEDs:LED_0805" H 3300 3500 50  0001 C CNN
-F 3 "" H 3300 3500 50  0000 C CNN
-	1    3300 3500
-	1    0    0    -1
-$EndComp
-$Comp
-L LED D21
-U 1 1 585D8AE5
-P 3300 3850
-AR Path="/585D8AE5" Ref="D21"  Part="1"
-AR Path="/585D6FEE/585D8AE5" Ref="D21"  Part="1"
-F 0 "D21" H 3300 3950 50  0000 C CNN
-F 1 "150060GS75000" H 3300 3750 50  0000 C CNN
-F 2 "LEDs:LED_0805" H 3300 3850 50  0001 C CNN
-F 3 "" H 3300 3850 50  0000 C CNN
-	1    3300 3850
-	1    0    0    -1
-$EndComp
-$Comp
-L LED D22
-U 1 1 585D8AEC
-P 3300 4200
-AR Path="/585D8AEC" Ref="D22"  Part="1"
-AR Path="/585D6FEE/585D8AEC" Ref="D22"  Part="1"
-F 0 "D22" H 3300 4300 50  0000 C CNN
-F 1 "150060GS75000" H 3300 4100 50  0000 C CNN
-F 2 "LEDs:LED_0805" H 3300 4200 50  0001 C CNN
-F 3 "" H 3300 4200 50  0000 C CNN
-	1    3300 4200
-	1    0    0    -1
-$EndComp
-$Comp
-L LED D23
-U 1 1 585D8AF3
-P 3300 4550
-AR Path="/585D8AF3" Ref="D23"  Part="1"
-AR Path="/585D6FEE/585D8AF3" Ref="D23"  Part="1"
-F 0 "D23" H 3300 4650 50  0000 C CNN
-F 1 "150060GS75000" H 3300 4450 50  0000 C CNN
-F 2 "LEDs:LED_0805" H 3300 4550 50  0001 C CNN
-F 3 "" H 3300 4550 50  0000 C CNN
-	1    3300 4550
-	1    0    0    -1
-$EndComp
-$Comp
 L LED D15
 U 1 1 585D8AFA
@@
 	1    0    0    -1
 $EndComp
-$Comp
-L LED D24
-U 1 1 585D8B16
-P 3300 4900
-AR Path="/585D8B16" Ref="D24"  Part="1"
-AR Path="/585D6FEE/585D8B16" Ref="D24"  Part="1"
-F 0 "D24" H 3300 5000 50  0000 C CNN
-F 1 "150060GS75000" H 3300 4800 50  0000 C CNN
-F 2 "LEDs:LED_0805" H 3300 4900 50  0001 C CNN
-F 3 "" H 3300 4900 50  0000 C CNN
-	1    3300 4900
-	1    0    0    -1
-$EndComp
 Text GLabel 2200 1650 2    60   Input ~ 0
 ROW1
 Text GLabel 2850 1650 2    60   Input ~ 0
 ROW2
-Text GLabel 3500 1650 2    60   Input ~ 0
-ROW3
 Text GLabel 1450 2650 0    60   Input ~ 0
 COL1
@@
 $EndComp
 $Comp
-L R-RESCUE-wnm_mk_1 R9
-U 1 1 5862A6DA
-P 3500 1900
-AR Path="/5862A6DA" Ref="R9"  Part="1"
-AR Path="/585D6FEE/5862A6DA" Ref="R9"  Part="1"
-F 0 "R9" V 3580 1900 40  0000 C CNN
-F 1 "330" V 3507 1901 40  0000 C CNN
-F 2 "Resistors_SMD:R_0805" V 3430 1900 30  0001 C CNN
-F 3 "" H 3500 1900 30  0000 C CNN
-	1    3500 1900
-	1    0    0    -1
-$EndComp
-$Comp
 L SSD1306 U9
 U 1 1 58642D78
@@
 Connection ~ 2850 3150
 Connection ~ 2850 3500
-Connection ~ 3500 3500
-Connection ~ 3500 3850
-Connection ~ 3500 4200
 Connection ~ 2200 4550
 Connection ~ 2200 4900
@@
 Connection ~ 2450 3000
 Wire Wire Line
-	3100 3500 3100 3700
-Connection ~ 3100 3700
-Wire Wire Line
 	1800 4550 1800 4750
 Connection ~ 1800 4750
@@
 Connection ~ 2450 3350
 Wire Wire Line
-	3100 4050 3100 3850
-Connection ~ 3100 4050
-Wire Wire Line
 	1800 4900 1800 5100
 Connection ~ 1800 5100
@@
 Connection ~ 2450 3700
 Wire Wire Line
-	3100 4400 3100 4200
-Connection ~ 3100 4400
-Wire Wire Line
 	1800 5250 1800 5450
 Connection ~ 1800 5450
@@
 	2450 4050 2450 3850
 Connection ~ 2450 4050
-Wire Wire Line
-	3100 4750 3100 4550
-Connection ~ 3100 4750
 Connection ~ 1800 2650
 Connection ~ 1800 3000
@@
 	2850 2150 2850 5250
 Connection ~ 2850 3850
-Wire Wire Line
-	3500 2150 3500 5250
-Connection ~ 3500 4550
-Connection ~ 3500 4900
-Connection ~ 3100 5100
 Connection ~ 2450 4400
-Wire Wire Line
-	3100 5100 3100 4900
 Connection ~ 2450 4750
-Wire Wire Line
-	1450 5100 3100 5100
-Wire Wire Line
-	1450 5450 3100 5450
-Wire Wire Line
-	3100 5450 3100 5250
-Wire Wire Line
-	3100 3700 1450 3700
-Wire Wire Line
-	1450 4050 3100 4050
-Wire Wire Line
-	1450 4400 3100 4400
-Wire Wire Line
-	1450 4750 3100 4750
 Connection ~ 2450 5100
 Connection ~ 2450 5450
@@
 P 6975 5150
 AR Path="/586468A3" Ref="#PWR031"  Part="1"
-AR Path="/585D6FEE/586468A3" Ref="#PWR034"  Part="1"
-F 0 "#PWR034" H 6975 5150 30  0001 C CNN
+AR Path="/585D6FEE/586468A3" Ref="#PWR028"  Part="1"
+F 0 "#PWR028" H 6975 5150 30  0001 C CNN
 F 1 "GND" H 6975 5080 30  0001 C CNN
 F 2 "" H 6975 5150 60  0001 C CNN
@@
 OLED screen
 Wire Wire Line
-	3100 5250 3150 5250
-Wire Wire Line
-	3500 5250 3450 5250
-Wire Wire Line
-	3500 4900 3450 4900
-Wire Wire Line
-	3100 4900 3150 4900
-Wire Wire Line
-	3100 4550 3150 4550
-Wire Wire Line
-	3450 4550 3500 4550
-Wire Wire Line
-	3500 4200 3450 4200
-Wire Wire Line
-	3100 4200 3150 4200
-Wire Wire Line
-	3100 3850 3150 3850
-Wire Wire Line
-	3450 3850 3500 3850
-Wire Wire Line
-	3500 3500 3450 3500
-Wire Wire Line
-	3150 3500 3100 3500
-Wire Wire Line
 	2850 2450 2800 2450
 Wire Wire Line
@@
 Wire Wire Line
 	2850 5250 2800 5250
+Wire Wire Line
+	1450 3700 2450 3700
+Wire Wire Line
+	1450 4050 2450 4050
+Wire Wire Line
+	1450 4400 2450 4400
+Wire Wire Line
+	1450 4750 2450 4750
+Wire Wire Line
+	1450 5100 2450 5100
+Wire Wire Line
+	1450 5450 2450 5450
 $EndSCHEMATC

Commit message: HW: Finish rev-D layout
Connections:
- net Screen_NReset renamed Screen_Nreset
Changed lines of the file:
@@
 3V3
 Text GLabel 8850 3825 0    60   Input ~ 0
-Screen_NReset
+Screen_Nreset
 Text GLabel 8850 4025 0    60   Input ~ 0
 Audio_SCL

Commit message: HW: rev D production files
Parts:
- D1, D10, D11, D12, D13, D14, D15, D16, D17, D2, D3, D4, D5, D6, D7, D8, D9: value 150060RS75000 -> red
- D18: value 150060GS75000 -> green
- R7, R8: value 330 -> 330ohm
Other:
- note added: "With 18 LEDs we could do a 4x5 (9 GPIOs) matrix, but having the LED logic\nmatrix following the placement layout produces a cleaner PCB. The trade-off is that we\nuse 3 more GPIOs."
- note removed: "With 24 LEDs we could do a 5x5 (10 GPIOs) matrix, but having the LED logic\nmatrix following the placement layout produces a cleaner PCB. The trade-off is that we\nuse 2 more GPIOs."
Changed lines of the file:
@@
 AR Path="/585D6FEE/585D8A6E" Ref="D10"  Part="1"
 F 0 "D10" H 2650 2550 50  0000 C CNN
-F 1 "150060RS75000" H 2650 2350 50  0000 C CNN
+F 1 "red" H 2650 2350 50  0000 C CNN
 F 2 "LEDs:LED_0805" H 2650 2450 50  0001 C CNN
 F 3 "" H 2650 2450 50  0000 C CNN
@@
 AR Path="/585D6FEE/585D8A75" Ref="D11"  Part="1"
 F 0 "D11" H 2650 2900 50  0000 C CNN
-F 1 "150060RS75000" H 2650 2700 50  0000 C CNN
+F 1 "red" H 2650 2700 50  0000 C CNN
 F 2 "LEDs:LED_0805" H 2650 2800 50  0001 C CNN
 F 3 "" H 2650 2800 50  0000 C CNN
@@
 AR Path="/585D6FEE/585D8A7C" Ref="D12"  Part="1"
 F 0 "D12" H 2650 3250 50  0000 C CNN
-F 1 "150060RS75000" H 2650 3050 50  0000 C CNN
+F 1 "red" H 2650 3050 50  0000 C CNN
 F 2 "LEDs:LED_0805" H 2650 3150 50  0001 C CNN
 F 3 "" H 2650 3150 50  0000 C CNN
@@
 AR Path="/585D6FEE/585D8A83" Ref="D13"  Part="1"
 F 0 "D13" H 2650 3600 50  0000 C CNN
-F 1 "150060RS75000" H 2650 3400 50  0000 C CNN
+F 1 "red" H 2650 3400 50  0000 C CNN
 F 2 "LEDs:LED_0805" H 2650 3500 50  0001 C CNN
 F 3 "" H 2650 3500 50  0000 C CNN
@@
 AR Path="/585D6FEE/585D8A8A" Ref="D14"  Part="1"
 F 0 "D14" H 2650 3950 50  0000 C CNN
-F 1 "150060RS75000" H 2650 3750 50  0000 C CNN
+F 1 "red" H 2650 3750 50  0000 C CNN
 F 2 "LEDs:LED_0805" H 2650 3850 50  0001 C CNN
 F 3 "" H 2650 3850 50  0000 C CNN
@@
 AR Path="/585D6FEE/585D8A91" Ref="D1"  Part="1"
 F 0 "D1" H 2000 2550 50  0000 C CNN
-F 1 "150060RS75000" H 2000 2350 50  0000 C CNN
+F 1 "red" H 2000 2350 50  0000 C CNN
 F 2 "LEDs:LED_0805" H 2000 2450 50  0001 C CNN
 F 3 "" H 2000 2450 50  0000 C CNN
@@
 AR Path="/585D6FEE/585D8A98" Ref="D2"  Part="1"
 F 0 "D2" H 2000 2900 50  0000 C CNN
-F 1 "150060RS75000" H 2000 2700 50  0000 C CNN
+F 1 "red" H 2000 2700 50  0000 C CNN
 F 2 "LEDs:LED_0805" H 2000 2800 50  0001 C CNN
 F 3 "" H 2000 2800 50  0000 C CNN
@@
 AR Path="/585D6FEE/585D8A9F" Ref="D3"  Part="1"
 F 0 "D3" H 2000 3250 50  0000 C CNN
-F 1 "150060RS75000" H 2000 3050 50  0000 C CNN
+F 1 "red" H 2000 3050 50  0000 C CNN
 F 2 "LEDs:LED_0805" H 2000 3150 50  0001 C CNN
 F 3 "" H 2000 3150 50  0000 C CNN
@@
 AR Path="/585D6FEE/585D8AA6" Ref="D4"  Part="1"
 F 0 "D4" H 2000 3600 50  0000 C CNN
-F 1 "150060RS75000" H 2000 3400 50  0000 C CNN
+F 1 "red" H 2000 3400 50  0000 C CNN
 F 2 "LEDs:LED_0805" H 2000 3500 50  0001 C CNN
 F 3 "" H 2000 3500 50  0000 C CNN
@@
 AR Path="/585D6FEE/585D8AAD" Ref="D5"  Part="1"
 F 0 "D5" H 2000 3950 50  0000 C CNN
-F 1 "150060RS75000" H 2000 3750 50  0000 C CNN
+F 1 "red" H 2000 3750 50  0000 C CNN
 F 2 "LEDs:LED_0805" H 2000 3850 50  0001 C CNN
 F 3 "" H 2000 3850 50  0000 C CNN
@@
 AR Path="/585D6FEE/585D8AB4" Ref="D6"  Part="1"
 F 0 "D6" H 2000 4300 50  0000 C CNN
-F 1 "150060RS75000" H 2000 4100 50  0000 C CNN
+F 1 "red" H 2000 4100 50  0000 C CNN
 F 2 "LEDs:LED_0805" H 2000 4200 50  0001 C CNN
 F 3 "" H 2000 4200 50  0000 C CNN
@@
 AR Path="/585D6FEE/585D8ABB" Ref="D7"  Part="1"
 F 0 "D7" H 2000 4650 50  0000 C CNN
-F 1 "150060RS75000" H 2000 4450 50  0000 C CNN
+F 1 "red" H 2000 4450 50  0000 C CNN
 F 2 "LEDs:LED_0805" H 2000 4550 50  0001 C CNN
 F 3 "" H 2000 4550 50  0000 C CNN
@@
 AR Path="/585D6FEE/585D8AC2" Ref="D8"  Part="1"
 F 0 "D8" H 2000 5000 50  0000 C CNN
-F 1 "150060RS75000" H 2000 4800 50  0000 C CNN
+F 1 "red" H 2000 4800 50  0000 C CNN
 F 2 "LEDs:LED_0805" H 2000 4900 50  0001 C CNN
 F 3 "" H 2000 4900 50  0000 C CNN
@@
 AR Path="/585D6FEE/585D8AC9" Ref="D9"  Part="1"
 F 0 "D9" H 2000 5350 50  0000 C CNN
-F 1 "150060RS75000" H 2000 5150 50  0000 C CNN
+F 1 "red" H 2000 5150 50  0000 C CNN
 F 2 "LEDs:LED_0805" H 2000 5250 50  0001 C CNN
 F 3 "" H 2000 5250 50  0000 C CNN
@@
 AR Path="/585D6FEE/585D8AFA" Ref="D15"  Part="1"
 F 0 "D15" H 2650 4300 50  0000 C CNN
-F 1 "150060RS75000" H 2650 4100 50  0000 C CNN
+F 1 "red" H 2650 4100 50  0000 C CNN
 F 2 "LEDs:LED_0805" H 2650 4200 50  0001 C CNN
 F 3 "" H 2650 4200 50  0000 C CNN
@@
 AR Path="/585D6FEE/585D8B01" Ref="D16"  Part="1"
 F 0 "D16" H 2650 4650 50  0000 C CNN
-F 1 "150060RS75000" H 2650 4450 50  0000 C CNN
+F 1 "red" H 2650 4450 50  0000 C CNN
 F 2 "LEDs:LED_0805" H 2650 4550 50  0001 C CNN
 F 3 "" H 2650 4550 50  0000 C CNN
@@
 AR Path="/585D6FEE/585D8B08" Ref="D17"  Part="1"
 F 0 "D17" H 2650 5000 50  0000 C CNN
-F 1 "150060RS75000" H 2650 4800 50  0000 C CNN
+F 1 "red" H 2650 4800 50  0000 C CNN
 F 2 "LEDs:LED_0805" H 2650 4900 50  0001 C CNN
 F 3 "" H 2650 4900 50  0000 C CNN
@@
 AR Path="/585D6FEE/585D8B0F" Ref="D18"  Part="1"
 F 0 "D18" H 2650 5350 50  0000 C CNN
-F 1 "150060GS75000" H 2650 5150 50  0000 C CNN
+F 1 "green" H 2650 5150 50  0000 C CNN
 F 2 "LEDs:LED_0805" H 2650 5250 50  0001 C CNN
 F 3 "" H 2650 5250 50  0000 C CNN
@@
 COL9
 Text Notes 1000 1500 0    60   ~ 0
-With 24 LEDs we could do a 5x5 (10 GPIOs) matrix, but having the LED logic\nmatrix following the placement layout produces a cleaner PCB. The trade-off is that we\nuse 2 more GPIOs.
+With 18 LEDs we could do a 4x5 (9 GPIOs) matrix, but having the LED logic\nmatrix following the placement layout produces a cleaner PCB. The trade-off is that we\nuse 3 more GPIOs.
 $Comp
 L R-RESCUE-wnm_mk_1 R7
@@
 AR Path="/585D6FEE/5862A3A6" Ref="R7"  Part="1"
 F 0 "R7" V 2280 1900 40  0000 C CNN
-F 1 "330" V 2207 1901 40  0000 C CNN
+F 1 "330ohm" V 2207 1901 40  0000 C CNN
 F 2 "Resistors_SMD:R_0805" V 2130 1900 30  0001 C CNN
 F 3 "" H 2200 1900 30  0000 C CNN
@@
 AR Path="/585D6FEE/5862A65F" Ref="R8"  Part="1"
 F 0 "R8" V 2930 1900 40  0000 C CNN
-F 1 "330" V 2857 1901 40  0000 C CNN
+F 1 "330ohm" V 2857 1901 40  0000 C CNN
 F 2 "Resistors_SMD:R_0805" V 2780 1900 30  0001 C CNN
 F 3 "" H 2850 1900 30  0000 C CNN
