File: hardware/Mk-I/micro-controller.sch (KiCad schematic (older format))
At the start: 37 parts, among them U10 STM32_SWD_Connector, U4 STM32F427VIT6, U8 Micro_SD_Card_Det_Hirose_DM3AT, X1 ABM3B-8.000MHZ-B2-T

Commit message: HW: Finish rev-D layout
Parts:
- removed TP_CMD1: TEST, Measurement_Points:Measurement_Point_Round-SMD-Pad_Small, symbol TEST
- renumbered TP_DAT3 to TP_DBG_RX1, TP_DAT2 to TP_DBG_TX1
Connections:
- net COL1: now also U4.34 (PC5/ETH_RMII_RX_D1/ETH_MII_RX_D1/EVENTOUT); no longer U4.15 (PC0/OTG_HS_ULPI_STP/EVENTOUT)
- net COL2: now also U4.36 (PB1/TIM3_CH4/TIM8_CH3N/OTG_HS_ULPI_D2/ETH_MII_RXD3/OTG_HS_INTN/TIM1_CH3N/EVENTOUT); no longer U4.17 (PC2/SPI2_MISO/OTG_HS_ULPI_DIR/ETH_MII_TXD2/I2S2ext_SD/EVENTOUT)
- net COL3: now also U4.39 (PE8/FSMC_D5/TIM1_CH1N/EVENTOUT); no longer U4.29 (PA4/SPI1_NSS/SPI3_NSS/USART2_CK/DCMI_HSYNC/OTG_HS_SOF/I2S3_WS/EVENTOUT)
- net COL4: now also U4.41 (PE10/FSMC_D7/TIM1_CH2N/EVENTOUT); no longer U4.35 (PB0/TIM3_CH3/TIM8_CH2N/OTG_HS_ULPI_D1/ETH_MII_RXD2/TIM1_CH2N/EVENTOUT)
- net COL5: now also U4.43 (PE12/FSMC_D9/TIM1_CH3N/EVENTOUT); no longer U4.40 (PE9/FSMC_D6/TIM1_CH1/EVENTOUT)
- net COL6: now also U4.45 (PE14/FSMC_D11/TIM1_CH4/EVENTOUT); no longer U4.44 (PE13/FSMC_D10/TIM1_CH3/EVENTOUT)
- net COL7: now also U4.47 (PB10/SPI2_SCK/I2S2_CK/I2C2_SCL/USART3_TX/OTG_HS_ULPI_D3/ETH_MII_RX_ER/TIM2_CH3/EVENTOUT); no longer U4.48 (PB11/I2C2_SDA/USART3_RX/OTG_HS_ULPI_D4/ETH_RMII_TX_EN/ETH_MII_TX_EN/TIM2_CH4/EVENTOUT)
- net COL8: now also U4.52 (PB13/SPI2_SCK/I2S2_CK/USART3_CTS/TIM1_CH1N/CAN2_TX/OTG_HS_ULPI_D6/ETH_RMII_TXD1/ETH_MII_TXD1/EVENTOUT); no longer U4.54 (PB15/SPI2_MOSI/I2S2_SD/TIM1_CH3N/TIM8_CH3N/TIM12_CH2/OTG_HS_DP/EVENTOUT)
- net COL9: now also U4.58 (PD11/FSMC_CLE/FSMC_A16/USART3_CTS/EVENTOUT); no longer U4.61 (PD14/FSMC_D0/TIM4_CH3/EVENTOUT/_EVENTOUT)
- net ENC_1_A: now also U4.32 (PA7/SPI1_MOSI/TIM8_CH1N/TIM14_CH1/TIM3_CH2/ETH_MII_RX_DV/TIM1_CH1N/RMII_CRS_DV/EVENTOUT); no longer U4.30 (PA5/SPI1_SCK/OTG_HS_ULPI_CK/TIM2_CH1_ETR/TIM8_CHIN/EVENTOUT)
- net ENC_1_B: now also U4.31 (PA6/SPI1_MISO/TIM8_BKIN/TIM13_CH1/DCMI_PIXCLK/TIM3_CH1/TIM1_BKIN/EVENTOUT); no longer U4.24 (PA1/USART2_RTS/UART4_RX/ETH_RMII_REF_CLK/ETH_MII_RX_CLK/TIM5_CH2/TIMM2_CH2/EVENTOUT)
- net ENC_2_A: now also U4.24 (PA1/USART2_RTS/UART4_RX/ETH_RMII_REF_CLK/ETH_MII_RX_CLK/TIM5_CH2/TIMM2_CH2/EVENTOUT); no longer U4.31 (PA6/SPI1_MISO/TIM8_BKIN/TIM13_CH1/DCMI_PIXCLK/TIM3_CH1/TIM1_BKIN/EVENTOUT)
- net ENC_2_B: now also U4.30 (PA5/SPI1_SCK/OTG_HS_ULPI_CK/TIM2_CH1_ETR/TIM8_CHIN/EVENTOUT); no longer U4.32 (PA7/SPI1_MOSI/TIM8_CH1N/TIM14_CH1/TIM3_CH2/ETH_MII_RX_DV/TIM1_CH1N/RMII_CRS_DV/EVENTOUT)
- net SD_DAT2: no longer TP_DBG_TX1.1
- net SD_DAT3: no longer TP_DBG_RX1.1
- net Screen_Nreset: now also U4.29 (PA4/SPI1_NSS/SPI3_NSS/USART2_CK/DCMI_HSYNC/OTG_HS_SOF/I2S3_WS/EVENTOUT); no longer U4.7 (PC13/EVENTOUT)
- net BUTTON_ROW3: now reaches U4.25 (PA2/USART2_TX/TIM5_CH3/TIM9_CH1/TIM2_CH3/ETH_MDIO/EVENTOUT)
- net BUTTON_COL1: now reaches U4.33 (PC4/ETH_RMII_RX_D0/ETH_MII_RX_D0/EVENTOUT)
- net BUTTON_COL3: now reaches U4.38 (PE7/FSMC_D4/TIM1_ETR/EVENTOUT)
- net BUTTON_COL5: now reaches U4.42 (PE11/FSMC_D8/TIM1_CH2/EVENTOUT)
- net BUTTON_COL7: now reaches U4.46 (PE15/FSMC_D12/TIM1_BKIN/EVENTOUT)
- net BUTTON_ROW1: now reaches U4.51 (PB12/SPI2_NSS/I2S2_WS/I2C2_SMBA/USART3_CK/TIM1_BKIN/CAN2_RX/OTG_HS_ULPI_D5/ETH_RMII_TXD0/ETH_MII_TXD0/OTG_HS_ID/EVENTOUT)
- net BUTTON_COL9: now reaches U4.53 (PB14/SPI2_MISO/TIM1_CH2N/TIM12_CH1/OTG_HS_DM/USART3_RTS/TIM8_CH2N/I2S2ext_SD/EVENTOUT)
- net DBG_TX: now reaches U4.55 (PD8/FSMC_D13/USART3_TX/EVENTOUT)
- net DBG_TX: now also TP_DBG_TX1.1
- net DBG_RX: now reaches U4.56 (PD9/FSMC_D14/USART3_RX/EVENTOUT)
- net DBG_RX: now also TP_DBG_RX1.1
- net BUTTON_COL11: now reaches U4.57 (PD10/FSMC_D15/USART3_CK/EVENTOUT)
- net B10: no longer names the net of U4.26 (PA3/USART2_RX/TIM5_CH4/TIM9_CH2/TIM2_CH4/OTG_HS_ULPI_D0/ETH_MII_COL/EVENTOUT)
- net ENC_1_SW: no longer names the net of U4.8 (PC14/OSC32_IN/EVENTOUT)
- net ENC_2_SW: no longer names the net of U4.9 (PC15/OSC32_OUT/EVENTOUT)
- net PLAY_WAKEUP renamed Play_WKUP
- net Write renamed FS_ID
- new net BUTTON_COL10: U4.54 (PB15/SPI2_MOSI/I2S2_SD/TIM1_CH3N/TIM8_CH3N/TIM12_CH2/OTG_HS_DP/EVENTOUT)
- new net BUTTON_COL2: U4.35 (PB0/TIM3_CH3/TIM8_CH2N/OTG_HS_ULPI_D1/ETH_MII_RXD2/TIM1_CH2N/EVENTOUT)
- new net BUTTON_COL4: U4.40 (PE9/FSMC_D6/TIM1_CH1/EVENTOUT)
- new net BUTTON_COL6: U4.44 (PE13/FSMC_D10/TIM1_CH3/EVENTOUT)
- new net BUTTON_COL8: U4.48 (PB11/I2C2_SDA/USART3_RX/OTG_HS_ULPI_D4/ETH_RMII_TX_EN/ETH_MII_TX_EN/TIM2_CH4/EVENTOUT)
- new net BUTTON_ROW2: U4.61 (PD14/FSMC_D0/TIM4_CH3/EVENTOUT/_EVENTOUT)
Other:
- moved on the sheet: TP_DBG_RX1, TP_DBG_TX1, U10
Changed lines of the file:
@@
 $EndComp
 Text GLabel 2850 4100 0    60   Input ~ 0
-PLAY_WAKEUP
+Play_WKUP
 $Comp
 L C-RESCUE-wnm_mk_1 C12
@@
 Text GLabel 12850 6700 2    60   Input ~ 0
 SD_DAT0
-Text GLabel 12850 5500 2    60   Input ~ 0
+Text GLabel 12850 5200 2    60   Input ~ 0
 COL9
 Text GLabel 12850 5400 2    60   Input ~ 0
@@
 Text GLabel 12850 5300 2    60   Input ~ 0
 ROW2
-Text GLabel 2850 7400 0    60   Input ~ 0
+Text GLabel 2850 7200 0    60   Input ~ 0
 COL8
-Text GLabel 2850 7000 0    60   Input ~ 0
+Text GLabel 2850 6900 0    60   Input ~ 0
 COL7
-Text GLabel 12850 3600 2    60   Input ~ 0
+Text GLabel 12850 3700 2    60   Input ~ 0
 COL6
-Text GLabel 12850 3200 2    60   Input ~ 0
+Text GLabel 12850 3500 2    60   Input ~ 0
 COL5
 Text GLabel 4950 9950 0    60   Input ~ 0
@@
 Text GLabel 12850 6900 2    60   Input ~ 0
 SD_DAT2
-Text GLabel 2850 5100 0    60   Input ~ 0
-Write
 Text GLabel 12850 7100 2    60   Input ~ 0
 SD_CLK
 Text GLabel 12850 4300 2    60   Input ~ 0
 SD_CMD
-Text GLabel 2850 5900 0    60   Input ~ 0
+Text GLabel 12850 3300 2    60   Input ~ 0
 COL4
-Text GLabel 2850 4500 0    60   Input ~ 0
+Text GLabel 12850 3100 2    60   Input ~ 0
 COL3
-Text GLabel 2850 4400 0    60   Input ~ 0
-B10
-Text GLabel 12850 6100 2    60   Input ~ 0
+Text GLabel 2850 6000 0    60   Input ~ 0
 COL2
-Text GLabel 12850 5900 2    60   Input ~ 0
+Text GLabel 12850 6400 2    60   Input ~ 0
 COL1
 $Comp
@@
 	1    0    0    -1
 $EndComp
+Text GLabel 2850 4800 0    60   Input ~ 0
+ENC_1_A
+Text GLabel 2850 4700 0    60   Input ~ 0
+ENC_1_B
+Text GLabel 2850 4200 0    60   Input ~ 0
+ENC_2_A
 Text GLabel 2850 4600 0    60   Input ~ 0
-ENC_1_A
-Text GLabel 2850 4200 0    60   Input ~ 0
-ENC_1_B
-Text GLabel 2850 4700 0    60   Input ~ 0
-ENC_2_A
-Text GLabel 2850 4800 0    60   Input ~ 0
 ENC_2_B
-Text GLabel 12850 7300 2    60   Input ~ 0
-ENC_1_SW
-Text GLabel 12850 7400 2    60   Input ~ 0
-ENC_2_SW
 $Comp
 L STM32_SWD_Connector U10
 U 1 1 58664887
-P 10250 9250
-F 0 "U10" H 10250 9250 60  0000 C CNN
-F 1 "STM32_SWD_Connector" V 10600 8600 60  0000 C CNN
-F 2 "stm32f4-disco:STM32_SWD_Connector_SMD" H 10250 9250 60  0001 C CNN
-F 3 "" H 10250 9250 60  0001 C CNN
-	1    10250 9250
-	1    0    0    -1
-$EndComp
-Text GLabel 10000 9400 0    60   Input ~ 0
+P 10250 8950
+F 0 "U10" H 10250 8950 60  0000 C CNN
+F 1 "STM32_SWD_Connector" V 10600 8300 60  0000 C CNN
+F 2 "stm32f4-disco:STM32_SWD_Connector_SMD" H 10250 8950 60  0001 C CNN
+F 3 "" H 10250 8950 60  0001 C CNN
+	1    10250 8950
+	1    0    0    -1
+$EndComp
+Text GLabel 10000 9100 0    60   Input ~ 0
 3V3
 $Comp
 L GND-RESCUE-wnm_mk_1 #PWR030
 U 1 1 586649ED
-P 9900 9850
+P 9900 9550
 AR Path="/586649ED" Ref="#PWR030"  Part="1"
 AR Path="/585DBE08/586649ED" Ref="#PWR022"  Part="1"
-F 0 "#PWR022" H 9900 9850 30  0001 C CNN
-F 1 "GND" H 9900 9780 30  0001 C CNN
-F 2 "" H 9900 9850 60  0001 C CNN
-F 3 "" H 9900 9850 60  0001 C CNN
-	1    9900 9850
-	1    0    0    -1
-$EndComp
-Text GLabel 10000 9600 0    60   Input ~ 0
+F 0 "#PWR022" H 9900 9550 30  0001 C CNN
+F 1 "GND" H 9900 9480 30  0001 C CNN
+F 2 "" H 9900 9550 60  0001 C CNN
+F 3 "" H 9900 9550 60  0001 C CNN
+	1    9900 9550
+	1    0    0    -1
+$EndComp
+Text GLabel 10000 9300 0    60   Input ~ 0
 SWCLK
-Text GLabel 10000 10000 0    60   Input ~ 0
+Text GLabel 10000 9700 0    60   Input ~ 0
 SWDIO
 Text GLabel 2000 2500 1    60   Input ~ 0
 NRST
-Text GLabel 10000 10200 0    60   Input ~ 0
+Text GLabel 10000 9900 0    60   Input ~ 0
 NRST
 Text GLabel 9100 1750 1    60   Input ~ 0
@@
 Text GLabel 2300 1800 2    60   Input ~ 0
 3V3
-Text GLabel 12850 7200 2    60   Input ~ 0
+Text GLabel 2850 4500 0    60   Input ~ 0
 Screen_Nreset
 Wire Wire Line
@@
 Connection ~ 5450 10250
 Wire Wire Line
-	9900 9850 9900 9800
-Wire Wire Line
-	9900 9800 10000 9800
+	9900 9550 9900 9500
+Wire Wire Line
+	9900 9500 10000 9500
 Wire Wire Line
 	2000 2500 2850 2500
@@
 Text GLabel 6900 10250 0    60   Input ~ 0
 SD_DETECT
-Text GLabel 3750 10150 0    60   Input ~ 0
-SD_DAT2
-Text GLabel 3750 10300 0    60   Input ~ 0
-SD_DAT3
-Text GLabel 3750 10450 0    60   Input ~ 0
-SD_CMD
+Text GLabel 10150 10650 0    60   Input ~ 0
+DBG_TX
+Text GLabel 10150 10800 0    60   Input ~ 0
+DBG_RX
 Text GLabel 3750 10750 0    60   Input ~ 0
 SD_DAT0
@@
 SD_DETECT
 $Comp
-L TEST TP_DAT2
+L TEST TP_DBG_TX1
 U 1 1 59EE5E47
-P 3750 10150
-F 0 "TP_DAT2" V 3750 10600 50  0000 C BNN
-F 1 "TEST" H 3750 10400 50  0000 C CNN
-F 2 "Measurement_Points:Measurement_Point_Round-SMD-Pad_Small" H 3750 10150 50  0001 C CNN
-F 3 "" H 3750 10150 50  0001 C CNN
-	1    3750 10150
-	0    1    1    0
-$EndComp
-$Comp
-L TEST TP_DAT3
+P 10150 10650
+F 0 "TP_DBG_TX1" V 10150 11200 50  0000 C BNN
+F 1 "TEST" H 10150 10900 50  0000 C CNN
+F 2 "Measurement_Points:Measurement_Point_Round-SMD-Pad_Small" H 10150 10650 50  0001 C CNN
+F 3 "" H 10150 10650 50  0001 C CNN
+	1    10150 10650
+	0    1    1    0
+$EndComp
+$Comp
+L TEST TP_DBG_RX1
 U 1 1 59EE61E0
-P 3750 10300
-F 0 "TP_DAT3" V 3800 10750 50  0000 C BNN
-F 1 "TEST" H 3750 10550 50  0000 C CNN
-F 2 "Measurement_Points:Measurement_Point_Round-SMD-Pad_Small" H 3750 10300 50  0001 C CNN
-F 3 "" H 3750 10300 50  0001 C CNN
-	1    3750 10300
-	0    1    1    0
-$EndComp
-$Comp
-L TEST TP_CMD1
-U 1 1 59EE6254
-P 3750 10450
-F 0 "TP_CMD1" V 3800 10900 50  0000 C BNN
-F 1 "TEST" H 3750 10700 50  0000 C CNN
-F 2 "Measurement_Points:Measurement_Point_Round-SMD-Pad_Small" H 3750 10450 50  0001 C CNN
-F 3 "" H 3750 10450 50  0001 C CNN
-	1    3750 10450
+P 10150 10800
+F 0 "TP_DBG_RX1" V 10200 11350 50  0000 C BNN
+F 1 "TEST" H 10150 11050 50  0000 C CNN
+F 2 "Measurement_Points:Measurement_Point_Round-SMD-Pad_Small" H 10150 10800 50  0001 C CNN
+F 3 "" H 10150 10800 50  0001 C CNN
+	1    10150 10800
 	0    1    1    0
 $EndComp
@@
 	0    1    1    0
 $EndComp
+Text GLabel 12850 5500 2    60   Input ~ 0
+BUTTON_ROW2
+Text GLabel 12850 5100 2    60   Input ~ 0
+BUTTON_COL11
+Text GLabel 2850 7400 0    60   Input ~ 0
+BUTTON_COL10
+Text GLabel 2850 7100 0    60   Input ~ 0
+BUTTON_ROW1
+Text GLabel 2850 7300 0    60   Input ~ 0
+BUTTON_COL9
+Text GLabel 2850 7000 0    60   Input ~ 0
+BUTTON_COL8
+Text GLabel 12850 3800 2    60   Input ~ 0
+BUTTON_COL7
+Text GLabel 12850 3600 2    60   Input ~ 0
+BUTTON_COL6
+Text GLabel 12850 3400 2    60   Input ~ 0
+BUTTON_COL5
+Text GLabel 12850 3200 2    60   Input ~ 0
+BUTTON_COL4
+Text GLabel 12850 6300 2    60   Input ~ 0
+BUTTON_COL1
+Text GLabel 2850 4300 0    60   Input ~ 0
+BUTTON_ROW3
+Text GLabel 12850 3000 2    60   Input ~ 0
+BUTTON_COL3
+Text GLabel 2850 5900 0    60   Input ~ 0
+BUTTON_COL2
+Text GLabel 12850 4900 2    60   Input ~ 0
+DBG_TX
+Text GLabel 12850 5000 2    60   Input ~ 0
+DBG_RX
+Text GLabel 2850 5100 0    60   Input ~ 0
+FS_ID
 $EndSCHEMATC

Commit message: HW: rev D production files
Parts:
- removed DFU_MODE1: Jumper_NO_Small, Buttons_Switches_SMD:SW_SPST_EVQP7A, symbol Jumper_NO_Small
- added DFU_MODE1: SW_PUSH, Buttons_Switches_SMD:SW_SPST_EVQP7A, symbol SW_PUSH
Connections:
- net 3V3: now also DFU_MODE1.1
- net BOOT0: now also DFU_MODE1.2
Changed lines of the file:
@@
 Text GLabel 2750 2300 1    60   Input ~ 0
 BOOT0
-$Comp
-L Jumper_NO_Small DFU_MODE1
-U 1 1 587582D9
-P 2200 1800
-F 0 "DFU_MODE1" H 2200 1950 50  0000 C CNN
-F 1 "Jumper_NO_Small" H 2250 1650 50  0000 C CNN
-F 2 "Buttons_Switches_SMD:SW_SPST_EVQP7A" H 2200 1800 50  0001 C CNN
-F 3 "" H 2200 1800 50  0000 C CNN
-	1    2200 1800
-	-1   0    0    1
-$EndComp
-Text GLabel 2100 1800 0    60   Input ~ 0
+Text GLabel 1900 1750 2    60   Input ~ 0
 BOOT0
-Text GLabel 2300 1800 2    60   Input ~ 0
+Text GLabel 1300 1750 0    60   Input ~ 0
 3V3
 Text GLabel 2850 4500 0    60   Input ~ 0
@@
 Text GLabel 2850 5100 0    60   Input ~ 0
 FS_ID
+$Comp
+L SW_PUSH DFU_MODE1
+U 1 1 59F72914
+P 1600 1750
+F 0 "DFU_MODE1" H 1750 1860 50  0000 C CNN
+F 1 "SW_PUSH" H 1600 1670 50  0000 C CNN
+F 2 "Buttons_Switches_SMD:SW_SPST_EVQP7A" H 1600 1750 60  0001 C CNN
+F 3 "" H 1600 1750 60  0000 C CNN
+	1    1600 1750
+	1    0    0    -1
+$EndComp
 $EndSCHEMATC
